File: aio-pcb-guide.kicad_pcb (KiCad board)
At the start: 2 copper layers, 24 parts, among them SW1 SW_Push, U1 ATmega32U4-AU, Y1 16MHz

Commit message: Some Routing Completed
Parts:
- C1, C2, C3, C4, C5, C6, C7, D1, D2, D3, D4, F1, R1, R2, R3, R4, SW1, U1, USB1, Y1: moved to B.Cu
- moved U1 90.9 mm to (124.6, 90.5), turned to 180 degrees
- moved C4 80.2 mm to (97.5, 94.5)
- moved C5 80.0 mm to (103.3, 94.5)
- moved C6 79.5 mm to (108.6, 94.5)
- moved C7 78.6 mm to (114.3, 94.5)
- moved R1 75.1 mm to (97.6, 81.0)
- moved R2 75.1 mm to (103.2, 81.0)
- moved R3 75.1 mm to (108.6, 81.0)
- moved R4 75.1 mm to (114.2, 81.0)
- moved F1 72.4 mm to (114.3, 74.6)
- moved Y1 68.8 mm to (124.6, 103.2), turned to 180 degrees
- moved C2 65.5 mm to (105.4, 88.1)
- moved C3 65.5 mm to (111.1, 88.1)
- moved SW1 57.8 mm to (180.2, 92.9)
- moved C1 41.5 mm to (119.9, 101.5), turned to 270 degrees
Connections:
- U1 pad 10: Net-(U1-Pad10) -> Col0
- U1 pad 11: Net-(U1-Pad11) -> Col1
- U1 pad 8: Net-(U1-Pad8) -> Row0
- U1 pad 9: Net-(U1-Pad9) -> Row1
Routing:
- net Col1: track 0.00 -> 54.6 mm, vias 0 -> 1
- net Row1: track 0.00 -> 51.0 mm
- net Row0: track 0.00 -> 38.1 mm
- net Col0: track 0.00 -> 33.1 mm, vias 0 -> 1
- net Net-(C1-Pad1): track 0.00 -> 18.1 mm
- net GND: track 0.00 -> 13.6 mm
- net Net-(D3-Pad2): track 0.00 -> 9.25 mm
- net Net-(D1-Pad2): track 0.00 -> 9.25 mm
- net Net-(D4-Pad2): track 0.00 -> 9.25 mm
- net Net-(D2-Pad2): track 0.00 -> 9.25 mm
- net Net-(C2-Pad1): track 0.00 -> 7.00 mm
