File: aio-pcb-guide.sch (KiCad schematic (older format))
At the start: 12 parts

Commit message: completed MCU
Parts:
- added R?: 10k, symbol Device:R_Small
- added SW?: SW_Push, symbol Switch:SW_Push
Connections:
- net labels added: D+, D-
- wire segments 57 -> 63
Other:
- moved on the sheet: C?, R?, U?, Y?

Commit message: Footprints applied
Parts:
- added D1, D2, D3, D4: D_Small, Diode_SMD:D_SOD-123, symbol Device:D_Small
- added F1: 500mA, Fuse:Fuse_1206_3216Metric, symbol Device:Fuse_Small
- added MX1, MX2, MX3, MX4: MX-NoLED, MX_Only:MXOnly-1U-NoLED, symbol MX_Alps_Hybrid:MX-NoLED
- added USB1: Molex-0548190589, random-keyboard-parts:Molex-0548190589, symbol random-keyboard-parts:Molex-0548190589
- C1, C2, C3, C4, C5, C6, C7: renamed from C?; footprint (none) -> Capacitor_SMD:C_0805_2012Metric
- R1, R2, R3, R4: renamed from R?; footprint (none) -> Resistor_SMD:R_0805_2012Metric
- SW1: renamed from SW?; footprint (none) -> random-keyboard-parts:SKQG-1155865
- Y1: renamed from Y?; footprint (none) -> Crystal:Crystal_SMD_3225-4Pin_3.2x2.5mm
- gave numbers to parts that had none: 1
Connections:
- net +5V: now also F1.2
- net D+: now also USB1.3 (D+)
- net D-: now also USB1.4 (D-)
- net GND: now also USB1.1 (GND)
- new net: D1.2 (A), MX1.2 (ROW)
- new net: D3.2 (A), MX3.2 (ROW)
- new net: D2.2 (A), MX2.2 (ROW)
- new net: D4.2 (A), MX4.2 (ROW)
- new net Col0: MX1.1 (COL), MX2.1 (COL)
- new net Col1: MX3.1 (COL), MX4.1 (COL)
- new net Row0: D1.1 (K), D3.1 (K)
- new net Row1: D2.1 (K), D4.1 (K)
- new net VCC: F1.1, USB1.5 (VBUS)
Other:
- moved on the sheet: C1, C2, C3, C4, C5, C6, C7, R1, R2, R3, R4, SW1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

Commit message: Some Routing Completed
Connections:
- net Col0: now also U1.10 (PB2)
- net Col1: now also U1.11 (PB3)
- net Row0: now also U1.8 (PB0)
- net Row1: now also U1.9 (PB1)
Changed lines of the file:
@@
 EESchema Schematic File Version 4
+LIBS:aio-pcb-guide-cache
 EELAYER 30 0
 EELAYER END
@@
 Wire Notes Line
 	5150 450  5150 3950
+Text GLabel 10350 1550 2    50   Input ~ 0
+Row0
+Text GLabel 10350 1650 2    50   Input ~ 0
+Row1
+Text GLabel 10350 1750 2    50   Input ~ 0
+Col0
+Text GLabel 10350 1850 2    50   Input ~ 0
+Col1
 $EndSCHEMATC
